File: Schematic/String-Drum-Synthesizer.kicad_pcb (KiCad board)
At the start: 2 copper layers, 62 parts, among them U1 LM1117MP-3.3, U2 SII1136CTU, U4 LM3900DR, U5 LM1117MP-3.3, U6 STM32F722RCTx

Commit message: Current Schem
Routing:
- net GND: track 0.00 -> 42.7 mm
- net +3V3: track 49.6 -> 71.6 mm
- net Net-(U5-GND): track 0.00 -> 16.5 mm
- net +5V: track 0.00 -> 16.1 mm
- net Net-(U1-GND): track 0.00 -> 9.78 mm
