File: Schematic/String-Drum-Synthesizer.kicad_sch (KiCad schematic)
At the start: 62 parts, among them U1 LM1117MP-3.3, U2 SII1136CTU, U3 74LS257, U4 LM3900DR, U5 LM1117MP-3.3, U6 STM32F722RCTx

Commit message: SCHEMATIC COMPLETE
Parts:
- removed R26: 1M, Resistor_THT:R_Axial_DIN0207_L6.3mm_D2.5mm_P7.62mm_Horizontal, symbol Device:R
- removed U3: 74LS257, Package_DIP:DIP-16_W7.62mm_Socket, symbol 74xx:74LS257
- added R33: 5.6k, Resistor_THT:R_Axial_DIN0207_L6.3mm_D2.5mm_P7.62mm_Horizontal, symbol Device:R
- R24: value 1M -> 4k7
- R25: value 1M -> 10k
Connections:
- net +5V: now also HDMI_Port1.18
- net GND: now also HDMI_Port1.11, HDMI_Port1.2, HDMI_Port1.5, HDMI_Port1.8, U2.10 (D8), U2.2 (D15), U2.3 (D14), U2.4 (D13), U2.6 (D12), U2.7 (D11), U2.78 (D35), U2.79 (D34), U2.8 (D10), U2.80 (D33), U2.81 (D32), U2.82 (D31), U2.83 (D30), U2.84 (D29), U2.85 (D28), U2.86 (D27), U2.87 (D26), U2.89 (D25), U2.9 (D9), U2.90 (D24), U2.92 (D23), U2.93 (D22), U2.94 (D21), U2.95 (D20), U2.96 (D19), U2.97 (D18), U2.98 (D17), U2.99 (D16), R33.2; no longer R24.1
- net PB2: no longer HDMI_Port1.7
- net PB3: no longer HDMI_Port1.9
- net PB4: no longer HDMI_Port1.4
- net PB5: no longer HDMI_Port1.6
- net PB6: no longer HDMI_Port1.1
- net PB7: no longer HDMI_Port1.3
- net PB8: now also U2.13 (D6)
- net PB9: now also U2.11 (D7)
- net HPD_OUT: now reaches U6.33 (PB12)
- net HPD_OUT: now also U2.76 (HPD)
- net IDCK: now reaches U2.22 (IDCK)
- net IDCK: now also U6.28 (PB10)
- net at U2.52 (EXT_SWING): now also R33.1
- net TXC-: now reaches U2.54 (TXC-)
- net TXC-: now also HDMI_Port1.12
- net TXC+: now reaches U2.55 (TXC+)
- net TXC+: now also HDMI_Port1.10
- net TX0-: now reaches U2.57 (TX0-)
- net TX0-: now also HDMI_Port1.9
- net TX0+: now reaches U2.58 (TX0+)
- net TX0+: now also HDMI_Port1.7
- net TX1-: now reaches U2.59 (TX1-)
- net TX1-: now also HDMI_Port1.6
- net TX1+: now reaches U2.60 (TX1+)
- net TX1+: now also HDMI_Port1.4
- net TX2-: now reaches U2.62 (TX2-)
- net TX2-: now also HDMI_Port1.3
- net TX2+: now reaches U2.63 (TX2+)
- net TX2+: now also HDMI_Port1.1
- net at HDMI_Port1.19: now also R24.2
- net HPD_IN: now reaches R25.2
- net HPD_IN: now also R24.1, U6.29 (PB11)
- net HDMI_PWR: no longer names the net of U6.50 (PA15)
- net HDMI_PWR: no longer HDMI_Port1.18
- net HDMI_PWR_SELECT: no longer names the net of U6.49 (PA14)
- removed net PB10: HDMI_Port1.10, U2.13 (D6), U6.28 (PB10)
- removed net PB11: HDMI_Port1.12, U2.11 (D7), U6.29 (PB11)
- net PC0 renamed DE
- net DE: now also U2.25 (DE); no longer U2.24 (HSYNC)
- net PC1 renamed HSYNC
- net HSYNC: now also U2.24 (HSYNC); no longer U2.23 (VSYNC)
- net PC13 renamed NRESET
- net PC2 renamed VSYNC
- net VSYNC: now also U2.23 (VSYNC); no longer U2.25 (DE)

Commit message: Half the copper traces work
Parts:
- added R26, R35: 10k, Resistor_THT:R_Axial_DIN0207_L6.3mm_D2.5mm_P7.62mm_Horizontal, symbol Device:R
- added R34: 5k6, Resistor_THT:R_Axial_DIN0207_L6.3mm_D2.5mm_P7.62mm_Horizontal, symbol Device:R
Connections:
- net +3.3V: now also R26.1, R35.2; no longer U2.16 (CVCC12__1), U2.21 (CVCC12__2), U2.38 (CVCC12__3), U2.5 (CVCC12), U2.56 (AVCC), U2.61 (AVCC__1), U2.88 (CVCC12__4)
- net DE: now also U6.34 (PB13); no longer U6.8 (PC0)
- net GND: now also R34.1
- net HSYNC: no longer names the net of U6.9 (PC1)
- net HSYNC: no longer U2.24 (HSYNC)
- net NRESET: no longer names the net of U6.2 (PC13)
- net NRESET: no longer U2.47 (~{RESET})
- net VSYNC: no longer names the net of U6.10 (PC2)
- net VSYNC: no longer U2.23 (VSYNC)
- new net: R34.2, R35.1, U2.16 (CVCC12__1), U2.21 (CVCC12__2), U2.38 (CVCC12__3), U2.5 (CVCC12), U2.56 (AVCC), U2.61 (AVCC__1), U2.88 (CVCC12__4)
- new net: R26.2, U2.47 (~{RESET})
Other:
- moved on the sheet: R15
